File: Power Supply.sch (KiCad schematic (older format))
At the start: 27 parts, among them J3 DC12V, U3 TPS563200, U4 TPS563200, U5 LP2985-1.8

Commit message: Rework: improving power delivery
Parts:
- added C18: 47u, Capacitor_SMD:C_1210_3225Metric_Pad1.42x2.65mm_HandSolder, symbol Device:C
- C10: renamed from C12; value 10µ -> 47µ; footprint Capacitor_SMD:C_0805_2012Metric_Pad1.15x1.40mm_HandSolder -> Capacitor_SMD:C_1210_3225Metric_Pad1.42x2.65mm_HandSolder
- C17: renamed from C13; value 47µ -> 220µ; footprint Capacitor_SMD:CP_Elec_5x5.3 -> Capacitor_Tantalum_SMD:CP_EIA-3528-12_Kemet-T_Pad1.50x2.35mm_HandSolder
- renumbered C14 to C11, C15 to C12, C7 to C13, C11 to C14, C16 to C15, C10 to C16, D6 to D4, D4 to D5, D5 to D6, R8 to R11, R10 to R12, R7 to R13, R9 to R14, R11 to R15, U3 to U4, U4 to U5, U5 to U6
Connections:
- wire segments 106 -> 110
Changed lines of the file:
@@
 $EndDescr
 $Comp
-L Regulator_Switching:TPS563200 U3
+L Regulator_Switching:TPS563200 U4
 U 1 1 5BA377A1
 P 5900 1800
-F 0 "U3" H 5900 2167 50  0000 C CNN
+F 0 "U4" H 5900 2167 50  0000 C CNN
 F 1 "TPS563200" H 5900 2076 50  0000 C CNN
 F 2 "Package_TO_SOT_SMD:SOT-23-6" H 5950 1550 50  0001 L CNN
@@
 $EndComp
 $Comp
-L Regulator_Switching:TPS563200 U4
+L Regulator_Switching:TPS563200 U5
 U 1 1 5BA377FD
 P 5900 3600
-F 0 "U4" H 5900 3967 50  0000 C CNN
+F 0 "U5" H 5900 3967 50  0000 C CNN
 F 1 "TPS563200" H 5900 3876 50  0000 C CNN
 F 2 "Package_TO_SOT_SMD:SOT-23-6" H 5950 3350 50  0001 L CNN
@@
 $EndComp
 $Comp
-L Regulator_Linear:LP2985-1.8 U5
+L Regulator_Linear:LP2985-1.8 U6
 U 1 1 5BA37A39
 P 5900 5500
-F 0 "U5" H 5900 5842 50  0000 C CNN
+F 0 "U6" H 5900 5842 50  0000 C CNN
 F 1 "LP2985-1.8" H 5900 5751 50  0000 C CNN
 F 2 "Package_TO_SOT_SMD:SOT-23-5" H 5900 5825 50  0001 C CNN
@@
 $EndComp
 $Comp
-L power:GND #PWR024
+L power:GND #PWR030
 U 1 1 5BA43606
 P 5900 2500
-F 0 "#PWR024" H 5900 2250 50  0001 C CNN
+F 0 "#PWR030" H 5900 2250 50  0001 C CNN
 F 1 "GND" H 5905 2327 50  0000 C CNN
 F 2 "" H 5900 2500 50  0001 C CNN
@@
 $EndComp
 $Comp
-L power:+12V #PWR022
+L power:+12V #PWR025
 U 1 1 5BA4364E
 P 3900 1600
-F 0 "#PWR022" H 3900 1450 50  0001 C CNN
+F 0 "#PWR025" H 3900 1450 50  0001 C CNN
 F 1 "+12V" H 3915 1773 50  0000 C CNN
 F 2 "" H 3900 1600 50  0001 C CNN
@@
 $EndComp
 $Comp
-L Device:C C7
+L Device:C C13
 U 1 1 5BA44F08
 P 6600 1550
-F 0 "C7" H 6715 1596 50  0000 L CNN
+F 0 "C13" H 6715 1596 50  0000 L CNN
 F 1 "100n" H 6715 1505 50  0000 L CNN
 F 2 "Capacitor_SMD:C_0603_1608Metric_Pad1.05x0.95mm_HandSolder" H 6638 1400 50  0001 C CNN
@@
 $EndComp
 $Comp
-L Device:R R7
+L Device:R R13
 U 1 1 5BA44FC1
 P 6750 1900
-F 0 "R7" V 6543 1900 50  0000 C CNN
+F 0 "R13" V 6543 1900 50  0000 C CNN
 F 1 "11k" V 6634 1900 50  0000 C CNN
 F 2 "Resistor_SMD:R_0603_1608Metric_Pad1.05x0.95mm_HandSolder" V 6680 1900 50  0001 C CNN
@@
 	6600 1300 7000 1300
 $Comp
-L Device:R R8
+L Device:R R11
 U 1 1 5BA45AA5
 P 6400 2150
-F 0 "R8" H 6470 2196 50  0000 L CNN
+F 0 "R11" H 6470 2196 50  0000 L CNN
 F 1 "2k" H 6470 2105 50  0000 L CNN
 F 2 "Resistor_SMD:R_0603_1608Metric_Pad1.05x0.95mm_HandSolder" V 6330 2150 50  0001 C CNN
@@
 $EndComp
 $Comp
-L Device:CP C10
+L Device:CP C16
 U 1 1 5BA45B25
 P 7000 2150
-F 0 "C10" H 7118 2196 50  0000 L CNN
+F 0 "C16" H 7118 2196 50  0000 L CNN
 F 1 "220µ" H 7118 2105 50  0000 L CNN
 F 2 "Capacitor_SMD:CP_Elec_6.3x5.3" H 7038 2000 50  0001 C CNN
@@
 $EndComp
 $Comp
-L power:+5V #PWR023
+L power:+5V #PWR034
 U 1 1 5BA45B82
 P 7100 1900
-F 0 "#PWR023" H 7100 1750 50  0001 C CNN
+F 0 "#PWR034" H 7100 1750 50  0001 C CNN
 F 1 "+5V" V 7115 2028 50  0000 L CNN
 F 2 "" H 7100 1900 50  0001 C CNN
@@
 	6400 2400 7000 2400
 $Comp
-L Device:C C12
+L Device:C C10
 U 1 1 5BA560B2
 P 5100 3750
-F 0 "C12" H 5215 3796 50  0000 L CNN
-F 1 "10µ" H 5215 3705 50  0000 L CNN
-F 2 "Capacitor_SMD:C_0805_2012Metric_Pad1.15x1.40mm_HandSolder" H 5138 3600 50  0001 C CNN
+F 0 "C10" H 5215 3796 50  0000 L CNN
+F 1 "47µ" H 5215 3705 50  0000 L CNN
+F 2 "Capacitor_SMD:C_1210_3225Metric_Pad1.42x2.65mm_HandSolder" H 5138 3600 50  0001 C CNN
 F 3 "~" H 5100 3750 50  0001 C CNN
 	1    5100 3750
@@
 $EndComp
 $Comp
-L Device:D_Schottky D4
+L Device:D_Schottky D5
 U 1 1 5BA5614D
 P 4850 3500
-F 0 "D4" H 4850 3716 50  0000 C CNN
+F 0 "D5" H 4850 3716 50  0000 C CNN
 F 1 "K34" H 4850 3625 50  0000 C CNN
 F 2 "Diode_SMD:D_SOD-123F" H 4850 3500 50  0001 C CNN
@@
 $EndComp
 $Comp
-L Device:C C11
+L Device:C C14
 U 1 1 5BA561C7
 P 6600 3350
-F 0 "C11" H 6715 3396 50  0000 L CNN
+F 0 "C14" H 6715 3396 50  0000 L CNN
 F 1 "100n" H 6715 3305 50  0000 L CNN
 F 2 "Capacitor_SMD:C_0603_1608Metric_Pad1.05x0.95mm_HandSolder" H 6638 3200 50  0001 C CNN
@@
 $EndComp
 $Comp
-L Device:R R10
+L Device:R R12
 U 1 1 5BA5629D
 P 6400 3950
-F 0 "R10" H 6470 3996 50  0000 L CNN
+F 0 "R12" H 6470 3996 50  0000 L CNN
 F 1 "10k" H 6470 3905 50  0000 L CNN
 F 2 "Resistor_SMD:R_0603_1608Metric_Pad1.05x0.95mm_HandSolder" V 6330 3950 50  0001 C CNN
@@
 $EndComp
 $Comp
-L Device:R R9
+L Device:R R14
 U 1 1 5BA56310
 P 6750 3700
-F 0 "R9" V 6543 3700 50  0000 C CNN
+F 0 "R14" V 6543 3700 50  0000 C CNN
 F 1 "33k" V 6634 3700 50  0000 C CNN
 F 2 "Resistor_SMD:R_0603_1608Metric_Pad1.05x0.95mm_HandSolder" V 6680 3700 50  0001 C CNN
@@
 $EndComp
 $Comp
-L Device:CP C13
+L Device:CP C17
 U 1 1 5BA563B8
 P 7000 3950
-F 0 "C13" H 7118 3996 50  0000 L CNN
-F 1 "47µ" H 7118 3905 50  0000 L CNN
-F 2 "Capacitor_SMD:CP_Elec_5x5.3" H 7038 3800 50  0001 C CNN
+F 0 "C17" H 7118 3996 50  0000 L CNN
+F 1 "220µ" H 7118 3905 50  0000 L CNN
+F 2 "Capacitor_Tantalum_SMD:CP_EIA-3528-12_Kemet-T_Pad1.50x2.35mm_HandSolder" H 7038 3800 50  0001 C CNN
 F 3 "~" H 7000 3950 50  0001 C CNN
 	1    7000 3950
@@
 $EndComp
 $Comp
-L power:+5V #PWR025
+L power:+5V #PWR028
 U 1 1 5BA56424
 P 5100 3400
-F 0 "#PWR025" H 5100 3250 50  0001 C CNN
+F 0 "#PWR028" H 5100 3250 50  0001 C CNN
 F 1 "+5V" H 5115 3573 50  0000 C CNN
 F 2 "" H 5100 3400 50  0001 C CNN
@@
 $EndComp
 $Comp
-L power:+3.3V #PWR027
+L power:+3.3V #PWR035
 U 1 1 5BA56538
-P 7700 3700
-F 0 "#PWR027" H 7700 3550 50  0001 C CNN
-F 1 "+3.3V" V 7715 3828 50  0000 L CNN
-F 2 "" H 7700 3700 50  0001 C CNN
-F 3 "" H 7700 3700 50  0001 C CNN
-	1    7700 3700
+P 8200 3700
+F 0 "#PWR035" H 8200 3550 50  0001 C CNN
+F 1 "+3.3V" V 8215 3828 50  0000 L CNN
+F 2 "" H 8200 3700 50  0001 C CNN
+F 3 "" H 8200 3700 50  0001 C CNN
+	1    8200 3700
 	0    1    1    0
 $EndComp
@@
 	6900 3700 7000 3700
 $Comp
-L power:GND #PWR028
+L power:GND #PWR031
 U 1 1 5BA5B7F2
 P 5900 4300
-F 0 "#PWR028" H 5900 4050 50  0001 C CNN
+F 0 "#PWR031" H 5900 4050 50  0001 C CNN
 F 1 "GND" H 5905 4127 50  0000 C CNN
 F 2 "" H 5900 4300 50  0001 C CNN
@@
 	4600 3500 4700 3500
 $Comp
-L Device:C C14
+L Device:C C11
 U 1 1 5BA65EC6
 P 5300 5750
-F 0 "C14" H 5415 5796 50  0000 L CNN
+F 0 "C11" H 5415 5796 50  0000 L CNN
 F 1 "10µ" H 5415 5705 50  0000 L CNN
 F 2 "Capacitor_SMD:C_0805_2012Metric_Pad1.15x1.40mm_HandSolder" H 5338 5600 50  0001 C CNN
@@
 $EndComp
 $Comp
-L Device:C C15
+L Device:C C12
 U 1 1 5BA65F36
 P 6400 5750
-F 0 "C15" H 6515 5796 50  0000 L CNN
+F 0 "C12" H 6515 5796 50  0000 L CNN
 F 1 "100n" H 6515 5705 50  0000 L CNN
 F 2 "Capacitor_SMD:C_0603_1608Metric_Pad1.05x0.95mm_HandSolder" H 6438 5600 50  0001 C CNN
@@
 $EndComp
 $Comp
-L Device:C C16
+L Device:C C15
 U 1 1 5BA65FF9
 P 6800 5750
-F 0 "C16" H 6915 5796 50  0000 L CNN
+F 0 "C15" H 6915 5796 50  0000 L CNN
 F 1 "10µ" H 6915 5705 50  0000 L CNN
 F 2 "Capacitor_SMD:C_0805_2012Metric_Pad1.15x1.40mm_HandSolder" H 6838 5600 50  0001 C CNN
@@
 $EndComp
 $Comp
-L power:+3.3V #PWR030
+L power:+3.3V #PWR029
 U 1 1 5BA66077
 P 5300 5300
-F 0 "#PWR030" H 5300 5150 50  0001 C CNN
+F 0 "#PWR029" H 5300 5150 50  0001 C CNN
 F 1 "+3.3V" H 5315 5473 50  0000 C CNN
 F 2 "" H 5300 5300 50  0001 C CNN
@@
 $EndComp
 $Comp
-L power:+1V8 #PWR031
+L power:+1V8 #PWR033
 U 1 1 5BA660EC
 P 6800 5300
-F 0 "#PWR031" H 6800 5150 50  0001 C CNN
+F 0 "#PWR033" H 6800 5150 50  0001 C CNN
 F 1 "+1V8" H 6815 5473 50  0000 C CNN
 F 2 "" H 6800 5300 50  0001 C CNN
@@
 Connection ~ 6800 5400
 $Comp
-L Diode:BAT54C D6
+L Diode:BAT54C D4
 U 1 1 5BA8AC6A
 P 4800 5500
-F 0 "D6" H 4800 5632 50  0000 C CNN
+F 0 "D4" H 4800 5632 50  0000 C CNN
 F 1 "BAT54C" H 4800 5723 50  0000 C CNN
 F 2 "Package_TO_SOT_SMD:SOT-23" H 4875 5625 50  0001 L CNN
@@
 	4300 5500 4300 5600
 $Comp
-L power:+BATT #PWR029
+L power:+BATT #PWR027
 U 1 1 5BA9237B
 P 4800 5200
-F 0 "#PWR029" H 4800 5050 50  0001 C CNN
+F 0 "#PWR027" H 4800 5050 50  0001 C CNN
 F 1 "+BATT" H 4815 5373 50  0000 C CNN
 F 2 "" H 4800 5200 50  0001 C CNN
@@
 	4800 5200 4800 5300
 $Comp
-L Device:LED D5
+L Device:LED D6
 U 1 1 5BADD32D
-P 7350 4200
-F 0 "D5" H 7341 4416 50  0000 C CNN
-F 1 "Power" H 7341 4325 50  0000 C CNN
-F 2 "LED_SMD:LED_0805_2012Metric_Pad1.15x1.40mm_HandSolder" H 7350 4200 50  0001 C CNN
-F 3 "~" H 7350 4200 50  0001 C CNN
-	1    7350 4200
-	1    0    0    -1
-$EndComp
-$Comp
-L Device:R R11
+P 7850 4200
+F 0 "D6" H 7841 4416 50  0000 C CNN
+F 1 "Power" H 7841 4325 50  0000 C CNN
+F 2 "LED_SMD:LED_0805_2012Metric_Pad1.15x1.40mm_HandSolder" H 7850 4200 50  0001 C CNN
+F 3 "~" H 7850 4200 50  0001 C CNN
+	1    7850 4200
+	1    0    0    -1
+$EndComp
+$Comp
+L Device:R R15
 U 1 1 5BADD3FC
-P 7600 3950
-F 0 "R11" H 7670 3996 50  0000 L CNN
-F 1 "510" H 7670 3905 50  0000 L CNN
-F 2 "Resistor_SMD:R_0603_1608Metric_Pad1.05x0.95mm_HandSolder" V 7530 3950 50  0001 C CNN
-F 3 "~" H 7600 3950 50  0001 C CNN
-	1    7600 3950
-	1    0    0    -1
-$EndComp
-Wire Wire Line
-	7000 3700 7600 3700
-Wire Wire Line
-	7600 3800 7600 3700
-Connection ~ 7600 3700
-Wire Wire Line
-	7600 3700 7700 3700
-Wire Wire Line
-	7500 4200 7600 4200
-Wire Wire Line
-	7600 4200 7600 4100
-Wire Wire Line
-	7000 4200 7200 4200
+P 8100 3950
+F 0 "R15" H 8170 3996 50  0000 L CNN
+F 1 "510" H 8170 3905 50  0000 L CNN
+F 2 "Resistor_SMD:R_0603_1608Metric_Pad1.05x0.95mm_HandSolder" V 8030 3950 50  0001 C CNN
+F 3 "~" H 8100 3950 50  0001 C CNN
+	1    8100 3950
+	1    0    0    -1
+$EndComp
+Wire Wire Line
+	8100 3800 8100 3700
+Connection ~ 8100 3700
+Wire Wire Line
+	8100 3700 8200 3700
+Wire Wire Line
+	8000 4200 8100 4200
+Wire Wire Line
+	8100 4200 8100 4100
 Connection ~ 7000 4200
+$Comp
+L Device:C C18
+U 1 1 5C13DB44
+P 7500 3950
+F 0 "C18" H 7615 3996 50  0000 L CNN
+F 1 "47u" H 7615 3905 50  0000 L CNN
+F 2 "Capacitor_SMD:C_1210_3225Metric_Pad1.42x2.65mm_HandSolder" H 7538 3800 50  0001 C CNN
+F 3 "~" H 7500 3950 50  0001 C CNN
+	1    7500 3950
+	1    0    0    -1
+$EndComp
+Wire Wire Line
+	7000 3700 7500 3700
+Wire Wire Line
+	7000 4200 7500 4200
+Wire Wire Line
+	7500 4100 7500 4200
+Connection ~ 7500 4200
+Wire Wire Line
+	7500 4200 7700 4200
+Wire Wire Line
+	7500 3800 7500 3700
+Connection ~ 7500 3700
+Wire Wire Line
+	7500 3700 8100 3700
 $EndSCHEMATC
