File: SushiBitsARMClassic.sch (KiCad schematic (older format))
At the start: 38 parts, among them J1 JTAG, J2 SPI, M1 LPC2103, P1 CONN_01X01, P2 CONN_01X01, P3 CONN_01X01, P4 CONN_01X01, P5 Digital, P6 Power, P7 Digital, P8 Analog, SW1 RESET, U1 MAX811S, U2 LMV321, U7 24LC512, Y1 32768, Y2 16M

Commit message: Rework: improving power delivery
Parts:
- P1: renamed from P6; footprint Socket_Arduino_Uno:Socket_Strip_Arduino_1x08 -> Connector_PinSocket_2.54mm:PinSocket_1x08_P2.54mm_Vertical
- P2: renamed from P8; footprint Socket_Arduino_Uno:Socket_Strip_Arduino_1x06 -> Connector_PinSocket_2.54mm:PinSocket_1x06_P2.54mm_Vertical
- P3: renamed from P5; footprint Socket_Arduino_Uno:Socket_Strip_Arduino_1x10 -> Connector_PinSocket_2.54mm:PinSocket_1x10_P2.54mm_Vertical
- P4: renamed from P7; footprint Socket_Arduino_Uno:Socket_Strip_Arduino_1x08 -> Connector_PinSocket_2.54mm:PinSocket_1x08_P2.54mm_Vertical
- SW1: footprint Button_Switch_SMD:SW_SPST_TL3305A -> Button_Switch_THT:SW_PUSH_6mm
- renumbered C19 to C5, C5 to C6, C6 to C7, J2 to J1, J1 to J2, P1 to P5, P2 to P6, P3 to P7, P4 to P8, R3 to R10, R14 to R3, R15 to R4, R6 to R5, R16 to R6, R5 to R7, R17 to R8, R4 to R9, U7 to U2, U2 to U3
Connections:
- wire segments 247 -> 251
