File: USBIF.sch (KiCad schematic (older format))
At the start: 12 parts, among them J4 USB_B, J5 Conn_ARM_JTAG_SWD_10, U6 STM32F042F4Px, Y3 16M

Commit message: Rework: improving power delivery
Parts:
- removed R13: 10k, Resistor_SMD:R_0603_1608Metric_Pad1.05x0.95mm_HandSolder, symbol Device:R
- renumbered C17 to C19, C18 to C20, R12 to R16, U6 to U7
Connections:
- net labels added: TCK, TDI, TDO, TMS
- no-connect marks 5 -> 2
Changed lines of the file:
@@
 $EndComp
 $Comp
-L MCU_ST_STM32F0:STM32F042F4Px U6
+L MCU_ST_STM32F0:STM32F042F4Px U7
 U 1 1 5BA79551
 P 6100 3100
-F 0 "U6" H 6100 2300 50  0000 C CNN
+F 0 "U7" H 6100 2300 50  0000 C CNN
 F 1 "STM32F042F4Px" H 6300 2200 50  0000 C CNN
 F 2 "Package_SO:TSSOP-20_4.4x6.5mm_P0.65mm" H 5600 2400 50  0001 R CNN
@@
 $EndComp
 $Comp
-L Device:C C18
+L Device:C C20
 U 1 1 5BA796F2
 P 8300 3950
-F 0 "C18" H 8415 3996 50  0000 L CNN
+F 0 "C20" H 8415 3996 50  0000 L CNN
 F 1 "100n" H 8415 3905 50  0000 L CNN
 F 2 "Capacitor_SMD:C_0603_1608Metric_Pad1.05x0.95mm_HandSolder" H 8338 3800 50  0001 C CNN
@@
 $EndComp
 $Comp
-L Device:C C17
+L Device:C C19
 U 1 1 5BA7973D
 P 7900 3950
-F 0 "C17" H 8015 3996 50  0000 L CNN
+F 0 "C19" H 8015 3996 50  0000 L CNN
 F 1 "100n" H 8015 3905 50  0000 L CNN
 F 2 "Capacitor_SMD:C_0603_1608Metric_Pad1.05x0.95mm_HandSolder" H 7938 3800 50  0001 C CNN
@@
 $EndComp
 $Comp
-L Device:R R12
+L Device:R R16
 U 1 1 5BA7979B
 P 6550 2300
-F 0 "R12" V 6343 2300 50  0000 C CNN
+F 0 "R16" V 6343 2300 50  0000 C CNN
 F 1 "10k" V 6434 2300 50  0000 C CNN
 F 2 "Resistor_SMD:R_0603_1608Metric_Pad1.05x0.95mm_HandSolder" V 6480 2300 50  0001 C CNN
@@
 	1    6550 2300
 	0    1    1    0
-$EndComp
-$Comp
-L Device:R R13
-U 1 1 5BA797EB
-P 6800 3950
-F 0 "R13" H 6870 3996 50  0000 L CNN
-F 1 "10k" H 6870 3905 50  0000 L CNN
-F 2 "Resistor_SMD:R_0603_1608Metric_Pad1.05x0.95mm_HandSolder" V 6730 3950 50  0001 C CNN
-F 3 "~" H 6800 3950 50  0001 C CNN
-	1    6800 3950
-	1    0    0    -1
 $EndComp
 $Comp
@@
 $EndComp
 $Comp
-L power:+3.3V #PWR034
+L power:+3.3V #PWR040
 U 1 1 5BA85390
 P 6200 2200
-F 0 "#PWR034" H 6200 2050 50  0001 C CNN
+F 0 "#PWR040" H 6200 2050 50  0001 C CNN
 F 1 "+3.3V" H 6215 2373 50  0000 C CNN
 F 2 "" H 6200 2200 50  0001 C CNN
@@
 $EndComp
 $Comp
-L power:GND #PWR037
+L power:GND #PWR041
 U 1 1 5BA857A0
 P 7400 4300
-F 0 "#PWR037" H 7400 4050 50  0001 C CNN
+F 0 "#PWR041" H 7400 4050 50  0001 C CNN
 F 1 "GND" H 7405 4127 50  0000 C CNN
 F 2 "" H 7400 4300 50  0001 C CNN
@@
 	7400 4100 7400 4200
 Wire Wire Line
-	7400 4200 6800 4200
-Wire Wire Line
 	6300 4200 6300 3900
 Connection ~ 7400 4200
@@
 	7400 4200 7400 4300
 Wire Wire Line
-	6800 4100 6800 4200
-Connection ~ 6800 4200
-Wire Wire Line
-	6800 4200 6300 4200
-Wire Wire Line
-	6700 3700 6800 3700
-Wire Wire Line
-	6800 3700 6800 3800
-Wire Wire Line
 	6700 3400 7100 3400
 Wire Wire Line
@@
 	7700 3900 7550 3900
 $Comp
-L power:VBUS #PWR035
+L power:VBUS #PWR039
 U 1 1 5BA86223
 P 4800 3200
-F 0 "#PWR035" H 4800 3050 50  0001 C CNN
+F 0 "#PWR039" H 4800 3050 50  0001 C CNN
 F 1 "VBUS" V 4815 3328 50  0000 L CNN
 F 2 "" H 4800 3200 50  0001 C CNN
@@
 	7900 4200 8300 4200
 $Comp
-L power:+3.3V #PWR036
+L power:+3.3V #PWR042
 U 1 1 5BA8955E
 P 7900 3600
-F 0 "#PWR036" H 7900 3450 50  0001 C CNN
+F 0 "#PWR042" H 7900 3450 50  0001 C CNN
 F 1 "+3.3V" H 7915 3773 50  0000 C CNN
 F 2 "" H 7900 3600 50  0001 C CNN
@@
 $EndComp
 $Comp
-L power:+3.3V #PWR038
+L power:+3.3V #PWR036
 U 1 1 5BA95596
 P 4300 4500
-F 0 "#PWR038" H 4300 4350 50  0001 C CNN
+F 0 "#PWR036" H 4300 4350 50  0001 C CNN
 F 1 "+3.3V" H 4315 4673 50  0000 C CNN
 F 2 "" H 4300 4500 50  0001 C CNN
@@
 $EndComp
 $Comp
-L power:GND #PWR039
+L power:GND #PWR037
 U 1 1 5BA955E4
 P 4300 6000
-F 0 "#PWR039" H 4300 5750 50  0001 C CNN
+F 0 "#PWR037" H 4300 5750 50  0001 C CNN
 F 1 "GND" H 4305 5827 50  0000 C CNN
 F 2 "" H 4300 6000 50  0001 C CNN
@@
 Wire Wire Line
 	5300 3100 5500 3100
-NoConn ~ 6700 3600
-NoConn ~ 5500 3300
-NoConn ~ 5500 3200
 $Comp
 L Device:LED D8
@@
 $EndComp
 $Comp
-L power:+3.3V #PWR033
+L power:+3.3V #PWR038
 U 1 1 5BAD371B
 P 4600 1900
-F 0 "#PWR033" H 4600 1750 50  0001 C CNN
+F 0 "#PWR038" H 4600 1750 50  0001 C CNN
 F 1 "+3.3V" H 4615 2073 50  0000 C CNN
 F 2 "" H 4600 1900 50  0001 C CNN
@@
 Wire Wire Line
 	4200 2700 4200 2400
+Wire Wire Line
+	6300 4200 7400 4200
+Text HLabel 5400 3200 0    50   Input ~ 0
+TDI
+Text HLabel 5400 3300 0    50   Input ~ 0
+TDO
+Text HLabel 6800 3600 2    50   Input ~ 0
+TCK
+Text HLabel 6800 3700 2    50   Input ~ 0
+TMS
+Wire Wire Line
+	5400 3200 5500 3200
+Wire Wire Line
+	5500 3300 5400 3300
+Wire Wire Line
+	6800 3600 6700 3600
+Wire Wire Line
+	6700 3700 6800 3700
 $EndSCHEMATC
